File: H0FR10/Design/H0FR10.brd (EAGLE design)
At the start: 34.6 x 30 mm, 26 parts, among them J1 CON-PHOENIX-350_1755749, K1 G5LE-14_DC3, P1 HEXABIT_17.32_NO_P6, Q1 MMBT3904LT1, U1 STM32F091CBU6, X1 XTALL_CSTCE8M00G52

Commit message: editing notes & descriptions (3oz to 2oz  & 10A to 8A)
Other:
- board text added: "30VDC/8A"
- board text added: "Note: This module should be manufactured with 2oz copper to handle 8A current."
- board text removed: "30VDC/10A"
- board text removed: "Note: This module should be manufactured with 3oz copper to handle 10A current."
Changed lines of the file:
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@@
 <?xml version="1.0" encoding="utf-8"?>
 <!DOCTYPE eagle SYSTEM "eagle.dtd">
-<eagle version="9.3.0">
+<eagle version="9.6.0">
 <drawing>
 <settings>
@@
 <rectangle x1="29.9107875" y1="23.887428125" x2="30.1317625" y2="23.902159375" layer="21"/>
 <rectangle x1="29.92551875" y1="23.9021625" x2="30.01390625" y2="23.91689375" layer="21"/>
-<text x="17.145" y="58.547" size="1.4224" layer="51">Note: This module should be manufactured with 3oz copper to handle 10A current.</text>
+<text x="17.145" y="58.547" size="1.4224" layer="51">Note: This module should be manufactured with 2oz copper to handle 8A current.</text>
 <rectangle x1="30.360871875" y1="20.1493125" x2="30.478728125" y2="20.16404375" layer="21"/>
 <rectangle x1="30.243015625" y1="20.16404375" x2="30.478728125" y2="20.178775" layer="21"/>
@@
 <rectangle x1="29.476953125" y1="20.267165625" x2="30.567121875" y2="20.281896875" layer="21"/>
 <rectangle x1="29.4474875" y1="20.2819" x2="30.56711875" y2="20.29663125" layer="21"/>
-<text x="40.767" y="47.117" size="1.6764" layer="22" rot="MR0">30VDC/10A</text>
+<text x="40.767" y="47.117" size="1.6764" layer="22" rot="MR0">30VDC/8A</text>
 <wire x1="32.004" y1="46.101" x2="32.004" y2="42.672" width="0.254" layer="22"/>
 <wire x1="32.004" y1="42.672" x2="36.957" y2="42.672" width="0.254" layer="22"/>

Commit message: Fix ERC errors Generate PDF Release at V0 again
Parts:
- R4: value 2400 Ω -> 1000 Ω
Changed lines of the file:
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@@
 <?xml version="1.0" encoding="utf-8"?>
 <!DOCTYPE eagle SYSTEM "eagle.dtd">
-<eagle version="9.6.0">
+<eagle version="9.6.1">
 <drawing>
 <settings>
@@
 <layer number="25" name="tNames" color="12" fill="1" visible="yes" active="yes"/>
 <layer number="26" name="bNames" color="9" fill="1" visible="yes" active="yes"/>
-<layer number="27" name="tValues" color="7" fill="1" visible="no" active="yes"/>
+<layer number="27" name="tValues" color="7" fill="1" visible="yes" active="yes"/>
 <layer number="28" name="bValues" color="7" fill="1" visible="no" active="yes"/>
 <layer number="29" name="tStop" color="7" fill="3" visible="no" active="yes"/>
@@
 <attribute name="VOLTAGE_RATING_DC" value="40.0 V" x="59.2582" y="2.1209" size="1.778" layer="28" rot="MR0" display="off"/>
 </element>
-<element name="R4" library="Hexabitz" package="R-0603" value="2400 Ω" x="34.70783125" y="29.08808125" smashed="yes" rot="MR270">
-<attribute name="MFN" value="Yageo" x="43.59783125" y="58.93308125" size="1.778" layer="28" rot="MR270" display="off"/>
-<attribute name="MPN" value="RC0603JR-070RL" x="43.59783125" y="58.93308125" size="1.778" layer="28" rot="MR270" display="off"/>
+<element name="R4" library="Hexabitz" package="R-0603" value="1000 Ω" x="34.70783125" y="29.08808125" smashed="yes" rot="MR270">
+<attribute name="MFN" value="Vishay" x="43.59783125" y="58.93308125" size="1.778" layer="28" rot="MR270" display="off"/>
+<attribute name="MPN" value="CRCW06031K00JNEA" x="43.59783125" y="58.93308125" size="1.778" layer="28" rot="MR270" display="off"/>
 <attribute name="NAME" x="35.53916875" y="28.36595625" size="1.016" layer="26" rot="MR90"/>
-<attribute name="OCTOPART_URL" value="https://octopart.com/crcw06032k40jnea-vishay-40298967" x="43.59783125" y="58.93308125" size="1.778" layer="28" rot="MR270" display="off"/>
-<attribute name="RESISTANCE" value="2400.0 Ω" x="43.59783125" y="58.93308125" size="1.778" layer="28" rot="MR270" display="off"/>
+<attribute name="OCTOPART_URL" value="https://octopart.com/crcw06031k00jnea-vishay-55388219?r=sp" x="43.59783125" y="58.93308125" size="1.778" layer="28" rot="MR270" display="off"/>
+<attribute name="RESISTANCE" value="1000.0 Ω" x="43.59783125" y="58.93308125" size="1.778" layer="28" rot="MR270" display="off"/>
 <attribute name="TOLERANCE" value="±5%" x="43.59783125" y="58.93308125" size="1.778" layer="28" rot="MR270" display="off"/>
 <attribute name="VALUE" x="36.597846875" y="30.626053125" size="1.016" layer="28" rot="MR270"/>
@@
 <attribute name="MF" value="STMicroelectronics" x="33.9598" y="25.949909375" size="1.778" layer="28" rot="MR180" display="off"/>
 <attribute name="MP" value="BAT54JFILM" x="33.9598" y="25.949909375" size="1.778" layer="28" rot="MR180" display="off"/>
+<attribute name="NAME" x="34.714303125" y="26.61858125" size="0.88965" layer="26" ratio="11" rot="MR0"/>
 <attribute name="NAME" x="32.68978125" y="26.58491875" size="0.635009375" layer="34" ratio="10" rot="MR180"/>
-<attribute name="NAME" x="34.714303125" y="26.61858125" size="0.88965" layer="26" ratio="11" rot="MR0"/>
 <attribute name="PACKAGE" value="SOD-323 STMicroelectronics" x="33.9598" y="25.949909375" size="1.778" layer="28" rot="MR180" display="off"/>
 <attribute name="PRICE" value="None" x="33.9598" y="25.949909375" size="1.778" layer="28" rot="MR180" display="off"/>
