File: H0FR11/Design/H0FR11.sch (EAGLE design)
At the start: 26 parts, among them J1 CON-PHOENIX-350_1755749, K1 G5LE-14_DC3, P1 HEXABIT_17.32_NO_P6, Q1 MMBT3904LT1, U1 STM32F091CBU6, X1 XTALL_CSTCE8M00G52

Commit message: - Changed to Rev1; this revision is 1OZ /4AMP..
Other:
- note added: "4A SPDT Relay"
- note added: "H0FR1"
- note added: "H0FR11_Backend"
- note added: "H0FR11_Frontend"
- note removed: "0"
- note removed: "8A SPDT Relay"
- note removed: "H0FR10"
- note removed: "H0FR10_Backend"
- note removed: "H0FR10_Frontend"
Changed lines of the file:
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@@
 <?xml version="1.0" encoding="utf-8"?>
 <!DOCTYPE eagle SYSTEM "eagle.dtd">
-<eagle version="9.6.1">
+<eagle version="9.6.2">
 <drawing>
 <settings>
-<setting alwaysvectorfont="yes"/>
+<setting alwaysvectorfont="no"/>
 <setting verticaltext="up"/>
 </settings>
@@
 <text x="215.9" y="5.3848" size="1.9304" layer="100" font="vector">Sheet   of</text>
 <text x="199.4662" y="19.6342" size="1.9304" layer="100" font="vector">Title</text>
-<text x="180.9242" y="19.6342" size="1.9304" layer="102" font="vector">H0FR10</text>
-<text x="179.2478" y="11.2014" size="1.9304" layer="101" font="vector">8A SPDT Relay </text>
-<text x="206.3242" y="19.6342" size="1.9304" layer="101" font="vector">H0FR10_Backend</text>
+<text x="180.9242" y="19.6342" size="1.9304" layer="102" font="vector">H0FR1</text>
+<text x="179.2478" y="11.2014" size="1.9304" layer="101" font="vector">4A SPDT Relay </text>
+<text x="206.3242" y="19.6342" size="1.9304" layer="101" font="vector">H0FR11_Backend</text>
 <wire x1="168.91" y1="3.81" x2="168.91" y2="8.128" width="0.1524" layer="205"/>
 <wire x1="168.91" y1="8.128" x2="168.91" y2="18.288" width="0.1524" layer="205"/>
 <wire x1="168.91" y1="18.288" x2="168.91" y2="22.86" width="0.1524" layer="205"/>
 <text x="222.25" y="10.2108" size="1.9304" layer="101" font="vector">Letter</text>
-<text x="227.6602" y="14.7066" size="1.9304" layer="101" font="vector">0</text>
+<text x="227.6602" y="14.7066" size="1.9304" layer="101" font="vector">1</text>
 <text x="223.52" y="5.3848" size="1.9304" layer="101" font="vector">1</text>
 <text x="228.346" y="5.3848" size="1.9304" layer="101" font="vector">2</text>
@@
 <text x="215.9" y="5.3848" size="1.9304" layer="100" font="vector">Sheet   of</text>
 <text x="199.4662" y="19.6342" size="1.9304" layer="100" font="vector">Title</text>
-<text x="180.9242" y="19.6342" size="1.9304" layer="102" font="vector">H0FR10</text>
-<text x="179.2478" y="11.2014" size="1.9304" layer="101" font="vector">8A SPDT Relay </text>
-<text x="206.3242" y="19.6342" size="1.9304" layer="101" font="vector">H0FR10_Frontend</text>
+<text x="180.9242" y="19.6342" size="1.9304" layer="102" font="vector">H0FR1</text>
+<text x="179.2478" y="11.2014" size="1.9304" layer="101" font="vector">4A SPDT Relay </text>
+<text x="206.3242" y="19.6342" size="1.9304" layer="101" font="vector">H0FR11_Frontend</text>
 <wire x1="168.91" y1="3.81" x2="168.91" y2="8.128" width="0.1524" layer="205"/>
 <wire x1="168.91" y1="8.128" x2="168.91" y2="18.288" width="0.1524" layer="205"/>
 <wire x1="168.91" y1="18.288" x2="168.91" y2="22.86" width="0.1524" layer="205"/>
 <text x="222.25" y="10.2108" size="1.9304" layer="101" font="vector">Letter</text>
-<text x="227.6602" y="14.7066" size="1.9304" layer="101" font="vector">0</text>
+<text x="227.6602" y="14.7066" size="1.9304" layer="101" font="vector">1</text>
 <text x="223.52" y="5.3848" size="1.9304" layer="101" font="vector">2</text>
 <text x="228.346" y="5.3848" size="1.9304" layer="101" font="vector">2</text>
