File: H0FR1/Design/H0FR1.sch (EAGLE design)
At the start: 25 parts, among them J1 CON-PHOENIX-350_1755749, K1 G5LE-14_DC3, P1 HEXABIT_17.32_NO_P6, Q1 MMBT3904LT1, U1 STM32G0B1CEU6N, X1 XTALL_CSTCE8M00G52

Commit message: Design modification
Parts:
- added C1, C10: 100nF, HEXABITZ_RCLS:C-0402
- added C11, C12: 330nF, HEXABITZ_RCLS:B32922Q3334K000
- added C9: 100nF, HEXABITZ_RCLS:C-0603
- added D4: MMSZ4705T1G, HEXABITZ_RCLS:MMSZ4705T1G
- added D5: BOURNS_CDSOD323-T03SCBOURNS_CDSOD323-T03SC_0_0, HEXABITZ_RCLS:BOURNS_CDSOD323-T03SCBOURNS_CDSOD323-T03SC_0_0
- added R15: 10k, HEXABITZ_RCLS:R-0402
- added R7: 0.0R, HEXABITZ_RCLS:R-0603
- added R9: 150, HEXABITZ_RCLS:R-0402
- added TRIMBLE-LOGO1, TRIMBLE-LOGO2: HEXA-LOGO, HEXABITZ_USER_INTERFACE_PARTS:HEXA-LOGO
- added Z1, Z2: MMSZ5231BT3G, HEXABITZ_RCLS:MMSZ5231BT3G
- C2: device HEXABITZ_RCLS:C-0402 -> HEXABITZ_RCLS:C-0603-POL; CAPACITANCE (none) -> 1.00uF; MFN (none) -> Yageo; MPN (none) -> CC0805KKX7R7BB105; OCTOPART_URL (none) -> https://octopart.com/cc0805kkx7r7bb105-yageo-8376555?r=sp&s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; TOLERANCE (none) -> 10%; VOLTAGE_RATING (none) -> 16V
- C3: CAPACITANCE (none) -> 100nF; MFN (none) -> KEMET; MPN (none) -> C0603C104K8RACTU; OCTOPART_URL (none) -> https://octopart.com/c0603c104k8ractu-kemet-145075?r=sp&s=9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; TOLERANCE (none) -> 10%; VOLTAGE_RATING (none) -> 10V
- C4: device HEXABITZ_RCLS:C-0402 -> HEXABITZ_RCLS:C-0603-POL; CAPACITANCE (none) -> 4.7uF; MFN (none) -> Murata; MPN (none) -> GRM21BC81E475KA12L; OCTOPART_URL (none) -> https://octopart.com/grm21bc81e475ka12l-murata-10331911?r=s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; TOLERANCE (none) -> 10%; VOLTAGE_RATING (none) -> 25V
- C5: device HEXABITZ_RCLS:C-0402 -> HEXABITZ_RCLS:C-0603
- C6: value 100nF -> 4.7uF; device HEXABITZ_RCLS:C-0402 -> HEXABITZ_RCLS:C-0603-POL; CAPACITANCE (none) -> 4.7uF; MFN (none) -> Murata; MPN (none) -> GRM21BC81E475KA12L; OCTOPART_URL (none) -> https://octopart.com/grm21bc81e475ka12l-murata-10331911?r=s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; TOLERANCE (none) -> 10%; VOLTAGE_RATING (none) -> 25V
- C7: value 4.7uF -> 100nF; CAPACITANCE (none) -> 100nF; MFN (none) -> KEMET; MPN (none) -> C0603C104K8RACTU; OCTOPART_URL (none) -> https://octopart.com/c0603c104k8ractu-kemet-145075?r=sp&s=9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; TOLERANCE (none) -> 10%; VOLTAGE_RATING (none) -> 10V
- FB1: value FB-TDK_MMZ1608Y300B -> (none); device HEXABITZ_RCLS:FB-TDK_MMZ1608Y300B -> HEXABITZ_RCLS:FB-0603; MFN TDK -> (none); MPN MMZ1608Y300B -> (none); OCTOPART_URL https://octopart.com/mmz1608y300b-tdk-368280?r=sp&s=cd9_2ZE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 -> (none)
- Q1: value MMBT3904LT1 -> BSS123; device HEXABITZ_RCLS:MMBT3904LT1 -> HEXABITZ_RCLS:BSS123; MFN ON Semiconductor -> (none); MPN MMBT3904LT1G -> (none); OCTOPART_ID 0bb6c2bc2200d471 -> (none); OCTOPART_URL http://octopart.com/mmbt3904lt1g-on+semiconductor-3280 -> (none); POLARITY NPN -> (none); POWER_DISSIPATION 0.225 W -> (none); VOLTAGE_RATING_DC 40.0 V -> (none)
- R2: value 180.0 Ω -> 180
- R3: value 10K -> 10k; MFN (none) -> Yageo; MPN (none) -> RC0603JR-0710KL; OCTOPART_URL (none) -> https://octopart.com/search?q=RC0603JR-0710KL&start=0; RESISTANCE (none) -> 10.0K Ohm; TOLERANCE (none) -> 5%
- R4: value 1000 Ω -> 150; MFN Vishay -> Yageo; MPN CRCW06031K00JNEA -> RC0603JR-07680KL; OCTOPART_URL https://octopart.com/crcw06031k00jnea-vishay-55388219?r=sp -> https://octopart.com/rc0603jr-07680kl-yageo-40953169?r=sp; RESISTANCE 1000.0 Ω -> 680K Ohm; TOLERANCE ±5% -> 5%
- R5: value 10.0 Ω -> 330; device HEXABITZ_RCLS:R-0402 -> HEXABITZ_RCLS:R-US_R2512; MFN Vishay -> (none); MPN CRCW060310R0FKEB -> (none); OCTOPART_URL https://octopart.com/crcw060310r0fkeb-vishay-42507905?r=sp&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 -> (none); POWER (none) -> 1W; RESISTANCE 10 Ohm -> (none); TOLERANCE ±1% -> (none)
- R6: value 0.0R -> 330; device HEXABITZ_RCLS:R-0402 -> HEXABITZ_RCLS:R-US_R2512; MFN Yageo -> (none); MPN RC0603JR-070RL -> (none); OCTOPART_URL https://octopart.com/rc0603jr-070rl-yageo-1241539?r=sp&s=X2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 -> (none); POWER (none) -> 1W; RESISTANCE 0.0 Ohm -> (none)
- SWD: device pinhead:PINHD-1X3 -> HEXABITZ_CONNECTION_PARTS:PINHD-1X3SWD
Connections:
- net N$3 renamed LED_INDICATOR
- removed net N$10: J1.1, K1.N.C.
- removed net N$117: U1.PC13
- removed net N$13: J1.3, K1.COM
- removed net N$7: J1.2, K1.N.O.
- new net COMMON: J1.3, K1.COM, R5.1, R6.1
- new net N$12: C12.2, R6.2
- new net N$17: K1.COIL_2
- new net N$3: Q1.G, R15.1, R9.1, Z1.K
- new net N$9: C11.2, R5.2
- new net NORMALLY_CLOSED: C12.1, J1.1, K1.N.C.
- new net NORMALLY_OPENED: C11.1, J1.2, K1.N.O.
- new net RELAY_CONTROL: R9.2
- new net VREF: C1.1, C2.1
- net GND: now also D4.A, D5.C, Q1.S, R15.2, R7.1, Z2.K; no longer Q1.E, R6.1
- net N$1: now also Z1.A, Z2.A; no longer D3.A, K1.COIL_2, R5.2
- net N$11: now also C10.1, R4.1; no longer Q1.B, R4.2
- net N$15: now also C10.2, D3.A, D4.K, Q1.D; no longer Q1.C, R5.1
- net SSR: no longer R4.1
- net VDD: now also D5.A, FB1.1, R4.2; no longer FB1.2
- net VDDA: now also FB1.2; no longer C2.1, C7.1, FB1.1
- net VSSA: now also C1.2, R7.2; no longer C7.2, R6.2
Other:
- note added: "AO3400A MOSFET 40 mOhm @VGS=3.3V"
- note added: "Contact Rating 10A - 230V"
- note added: "Ningbo Songle Relay SRD-03VDC-SL-C"
- note added: "Note! check footprint"
- note added: "SPDT Relay"
- note added: "VDDA Coupling"
- note added: "Zener 18V 0.5W"
- note added: "Zener 5.1V 0.5W"
- note removed: "10A SPDT Relay"
- note removed: "VDD\VDDA Coupling"
- moved on the sheet: C3, C5, C7, C8, D1, D2, D3, FB1, J1, K1, R, R1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

Commit message: Schematic modification
Parts:
- removed C11, C12: 330nF, HEXABITZ_RCLS:B32922Q3334K000
- C10: value 100nF -> 330nF; device HEXABITZ_RCLS:C-0402 -> HEXABITZ_RCLS:B32922Q3334K000; CAPACITANCE 100nF -> (none); MFN KEMET -> (none); MPN C0603C104K8RACTU -> (none); OCTOPART_URL https://octopart.com/c0603c104k8ractu-kemet-145075?r=sp&s=9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 -> (none); TOLERANCE 10% -> (none); VOLTAAGE (none) -> 450V; VOLTAGE_RATING 10V -> (none)
- C7: CAPACITANCE 100nF -> (none); MFN KEMET -> (none); MPN C0603C104K8RACTU -> (none); OCTOPART_URL https://octopart.com/c0603c104k8ractu-kemet-145075?r=sp&s=9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 -> (none); TOLERANCE 10% -> (none); VOLTAGE_RATING 10V -> (none)
- C8: CAPACITANCE (none) -> 100nF; MFN (none) -> KEMET; MPN (none) -> C0603C104K8RACTU; OCTOPART_URL (none) -> https://octopart.com/c0603c104k8ractu-kemet-145075?r=sp&s=9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; TOLERANCE (none) -> 10%; VOLTAGE_RATING (none) -> 10V
- C9: value 100nF -> 330nF; device HEXABITZ_RCLS:C-0603 -> HEXABITZ_RCLS:B32922Q3334K000; VOLTAAGE (none) -> 450V
- renumbered K1 to U2, R15 to R8, Z1 to D6, Z2 to D7
Connections:
- removed net SSR: U1.PB6
- net GND: now also C7.2; no longer C8.2
- net N$11: now also C8.1; no longer C10.1
- net N$12: now also C10.2; no longer C12.2
- net N$15: now also C8.2; no longer C10.2
- net N$4: now also C7.1; no longer C8.1
- net N$9: now also C9.2; no longer C11.2
- net NORMALLY_CLOSED: now also C10.1; no longer C12.1
- net NORMALLY_OPENED: now also C9.1; no longer C11.1
- net RELAY_CONTROL: now also U1.PB6
- net VDD: no longer D2.A, D3.C, R4.2, U2.COIL_1
- net VDDA: now also D2.A, D3.C, R4.2, U2.COIL_1
Other:
- moved on the sheet: C7

Commit message: Edit the decription
Other:
- note added: "230V 10A(RMS) SPDT Relay"
- note removed: "SPDT Relay"
Changed lines of the file:
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@@
 <wire x1="231.013" y1="18.034" x2="231.013" y2="22.606" width="0.1524" layer="205"/>
 <text x="242.5192" y="5.9182" size="1.9304" layer="100" font="vector">www.hexabitz.com</text>
-<text x="184.2008" y="10.9474" size="1.9304" layer="101" font="vector">SPDT Relay</text>
+<text x="174.6758" y="10.9474" size="1.9304" layer="101" font="vector">230V 10A(RMS) SPDT Relay</text>
 <text x="241.935" y="139.065" size="1.778" layer="125">BOOT</text>
 <text x="187.96" y="85.725" size="1.778" layer="95">VDDIO2 Coupling</text>
@@
 <wire x1="231.013" y1="18.542" x2="231.013" y2="23.114" width="0.1524" layer="205"/>
 <text x="242.5192" y="6.4262" size="1.9304" layer="100" font="vector">www.hexabitz.com</text>
-<text x="184.2008" y="11.4554" size="1.9304" layer="101" font="vector">SPDT Relay</text>
+<text x="174.0408" y="11.4554" size="1.9304" layer="101" font="vector">230V 10A(RMS) SPDT Relay</text>
 <text x="144.145" y="126.365" size="2.54" layer="89" font="vector" ratio="11" distance="46">Contact Rating
 10A  - 230V</text>

Commit message: Intial parts placing on the board
Parts:
- removed C3: 100nF, HEXABITZ_RCLS:C-0402
- removed C4: 4.7uF, HEXABITZ_RCLS:C-0603-POL
- removed J1: CON-PHOENIX-350_1755749, Hexabitz:CON-PHOENIX-350_1755749
- removed TRIMBLE-LOGO1: HEXA-LOGO, HEXABITZ_USER_INTERFACE_PARTS:HEXA-LOGO
- added X2: (no value), HEXABITZ_CONNECTION_PARTS:AK300/3
- C1, C7, C8: device HEXABITZ_RCLS:C-0402 -> HEXABITZ_RCLS:C-0603
- C2, C6: device HEXABITZ_RCLS:C-0603-POL -> HEXABITZ_RCLS:C-0805
- D3: value SMD-DIODE-SCHOTTKY-40V-300MA(SOD-323) -> 40V 300MA; device Hexabitz:SMD-DIODE-SCHOTTKY-40V-300MA(SOD-323) -> HEXABITZ_RCLS:BAT54JFILM_SOD-323
- D4: value MMSZ4705T1G -> MMSZ4705T1GMMSZ4705T1G; device HEXABITZ_RCLS:MMSZ4705T1G -> HEXABITZ_RCLS:MMSZ4705T1GMMSZ4705T1G
- D6, D7: value MMSZ5231BT3G -> MMSZ4705T1GMMSZ4705T1G; device HEXABITZ_RCLS:MMSZ5231BT3G -> HEXABITZ_RCLS:MMSZ4705T1GMMSZ4705T1G
- P1: value HEXABIT_17.32_NO_P6 -> HEXABIT_X2_P1_P5_EDIT_POWER_PADS; device hexabitz_connectors:HEXABIT_17.32_NO_P6 -> hexabitz_connectors:HEXABIT_X2_P1_P5_EDIT_POWER_PADS
- R1, R2, R3, R4, R8, R9: device HEXABITZ_RCLS:R-0402 -> HEXABITZ_RCLS:R-0603
- R5, R6: MPN (none) -> RMCF2512JT330R
- U1: value STM32G0B1CEU6N -> STM32G0B1CEU6QFN_B1CEU6_STM-L; device HEXABITZ_ICs:STM32G0B1CEU6N -> HEXABITZ_ICs:STM32G0B1CEU6QFN_B1CEU6_STM-L
Connections:
- removed net N$17: U2.COIL_2
- removed net VREF: C1.1, C2.1
- net COMMON: now also X2-2.KL; no longer J1.3
- net GND: now also P1.GND7, P1.GND8; no longer C3.2, C4.2, U1.EPAD
- net N$15: now also D3.+, U2.COIL_2; no longer D3.A
- net NORMALLY_CLOSED: now also X2-3.KL; no longer J1.1
- net NORMALLY_OPENED: now also X2-1.KL; no longer J1.2
- net USART4_RX: no longer P1.SD1
- net USART4_TX: no longer P1.SU1
- net USART6_RX: now also P1.SD1, U1.PB8; no longer U1.PA5
- net USART6_TX: now also P1.SU1, U1.PB9; no longer U1.PA4
- net VDD: now also D2.A, D3.-, P1.VDD7, P1.VDD8, R4.2, U2.COIL_1; no longer C3.1, C4.1, U1.VDDIO2
- net VDDA: now also C1.1, C2.1; no longer D2.A, D3.C, R4.2, U2.COIL_1
Other:
- note removed: "AO3400A MOSFET 40 mOhm @VGS=3.3V"
- note removed: "Ningbo Songle Relay SRD-03VDC-SL-C"
- note removed: "Note! check footprint"
- note removed: "VDDIO2 Coupling"
- note removed: "Zener 18V 0.5W"
- note removed: "Zener 5.1V 0.5W"
- moved on the sheet: C1, C10, C5, C9, D5, FB1, R5, R6, R7
