File: Design/H0FR1.sch (EAGLE design)
At the start: 34 parts, among them P1 HEXABIT_X2_P1_P5_EDIT_POWER_P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, Q1 BSS123, U1 STM32G0B1CEU6QFN_B1CEU6_STM-L, U2 G5LE-14_DC3, X1 XTALL_CSTCE8M00G52

Commit message: All finish, reviewed version
Parts:
- removed C10, C9: 330nF, HEXABITZ_RCLS:B32922Q3334K000
- removed C2: 1uF, HEXABITZ_RCLS:C-0805
- removed C7: 100nF, HEXABITZ_RCLS:C-0603
- removed D4, D6, D7: MMSZ4705T1GMMSZ4705T1G, HEXABITZ_RCLS:MMSZ4705T1GMMSZ4705T1G
- removed Q1: BSS123, HEXABITZ_RCLS:BSS123
- removed R4: 150, HEXABITZ_RCLS:R-0603
- removed R5, R6: 330, HEXABITZ_RCLS:R-US_R2512
- removed TRIMBLE-LOGO2: HEXA-LOGO, HEXABITZ_USER_INTERFACE_PARTS:HEXA-LOGO
- added C3: 100nF, HEXABITZ_RCLS:C-0603
- added C4: 4.7uF, HEXABITZ_RCLS:C-0805
- added Q2: BSS123, HEXABITZ_RCLS:BSS123
- added R10: 150, HEXABITZ_RCLS:R-0603
- added TRIMBLE-LOGO1: HEXA-LOGO, HEXABITZ_USER_INTERFACE_PARTS:HEXA-LOGO
- C1: value 100nF -> 1uF; device HEXABITZ_RCLS:C-0603 -> HEXABITZ_RCLS:C-0805; CAPACITANCE 100nF -> (none); MFN KEMET -> (none); MPN C0603C104K8RACTU -> (none); OCTOPART_URL https://octopart.com/c0603c104k8ractu-kemet-145075?r=sp&s=9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 -> (none); TOLERANCE 10% -> (none); VOLTAGE_RATING 10V -> (none)
- C6: value 4.7uF -> 100nF; device HEXABITZ_RCLS:C-0805 -> HEXABITZ_RCLS:C-0603; CAPACITANCE 4.7uF -> (none); MFN Murata -> (none); MPN GRM21BC81E475KA12L -> (none); OCTOPART_URL https://octopart.com/grm21bc81e475ka12l-murata-10331911?r=s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 -> (none); TOLERANCE 10% -> (none); VOLTAGE_RATING 25V -> (none)
- D2: value RED -> orange; COULOR (none) -> ORANGE
- FB1: value (none) -> FB-TDK_MMZ1608Y300B; MFN (none) -> TDK; MPN (none) -> MMZ1608Y300B; OCTOPART_URL (none) -> https://octopart.com/mmz1608y300b-tdk-368280?r=sp&s=cd9_2ZE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
- P1: value HEXABIT_X2_P1_P5_EDIT_POWER_PADS -> HEXABIT_17.32_NO_P6; device hexabitz_connectors:HEXABIT_X2_P1_P5_EDIT_POWER_PADS -> hexabitz_connectors:HEXABIT_17.32_NO_P6
- R2: value 180 -> 180.0 Ω
- R3: value 10k -> 10K; MFN Yageo -> (none); MPN RC0603JR-0710KL -> (none); OCTOPART_URL https://octopart.com/search?q=RC0603JR-0710KL&start=0 -> (none); RESISTANCE 10.0K Ohm -> (none); TOLERANCE 5% -> (none)
- R7: MFN (none) -> Yageo; MPN (none) -> RC0603JR-070RL; OCTOPART_URL (none) -> https://octopart.com/rc0603jr-070rl-yageo-1241539?r=sp&s=X2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; RESISTANCE (none) -> 0.0 Ohm
- R9: MFN Yageo -> Vishay; MPN RC0603JR-07680KL -> CRCW06031K00JNEA; OCTOPART_URL https://octopart.com/rc0603jr-07680kl-yageo-40953169?r=sp -> https://octopart.com/crcw06031k00jnea-vishay-55388219?r=sp; RESISTANCE 680K Ohm -> 1000.0 Ω; TOLERANCE 5% -> ±5%
- SWD: device HEXABITZ_CONNECTION_PARTS:PINHD-1X3SWD -> pinhead:PINHD-1X3
- U1: SPICEPREFIX (none) -> X
Connections:
- removed net COMMON: R5.1, R6.1, U2.COM, X2-2.KL
- removed net LED_INDICATOR: D1.A, U1.PA6
- removed net N$15: C8.2, D3.+, D4.K, Q1.D, R2.1, U2.COIL_2
- removed net N$9: C9.2, R5.2
- removed net NORMALLY_CLOSED: C10.1, U2.N.C., X2-3.KL
- removed net NORMALLY_OPENED: C9.1, U2.N.O., X2-1.KL
- removed net USART4_RX: U1.PA1
- removed net USART4_TX: U1.PA0
- new net COM: U2.COM, X2-3.KL
- new net NC: U2.N.C., X2-1.KL
- new net NO: U2.N.O., X2-2.KL
- new net USART1_RX: P1.SD5, U1.PB7
- new net USART1_TX: P1.SU5, U1.PB6
- net GND: now also C3.2, D1.C, D5.A, Q2.S; no longer C7.2, D4.A, D5.C, D7.K, P1.GND7, P1.GND8, Q1.S, R1.2
- net N$1: now also C8.2, D3.+, Q2.D, R2.1, U2.COIL_2; no longer D6.A, D7.A
- net N$11: now also Q2.G, R8.1, R9.2; no longer C8.1, R4.1
- net N$12: now also C8.1, R10.1; no longer C10.2, R6.2
- net N$2: now also D1.A, R1.2; no longer D1.C, R1.1
- net N$3: now also R1.1, U1.PA6; no longer D6.K, Q1.G, R8.1, R9.1
- net N$4: now also C3.1; no longer C7.1
- net RELAY_CONTROL: now also R9.1, U1.PB5; no longer R9.2, U1.PB6
- net USART5_RX: now also P1.SD3, U1.PB1; no longer P1.SD5, U1.PD2
- net USART5_TX: now also P1.SU3, U1.PB0; no longer P1.SU5, U1.PD3
- net USART6_RX: now also U1.PB9; no longer P1.SD3, U1.PB8
- net USART6_TX: now also U1.PB8; no longer P1.SU3, U1.PB9
- net VDD: now also D5.C, FB1.2, R10.2; no longer D5.A, FB1.1, P1.VDD7, P1.VDD8, R4.2
- net VDDA: now also C4.1, FB1.1; no longer C2.1, FB1.2
- net VSSA: now also C4.2; no longer C2.2
Other:
- note added: "230V/10A (RMS) SPDT Relay"
- note added: "VDD\VDDA Coupling"
- note removed: "230V 10A(RMS) SPDT Relay"
- note removed: "Contact Rating 10A - 230V"
- note removed: "VDDA Coupling"
- moved on the sheet: C1, C5, C6, C8, D1, D2, D3, D5, FB1, R, R1, R2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
